Commit message: Update init/shutdown sequences and urdf

File: urdf/ieg76.urdf.xacro (robot description, xacro)
@@ -1,12 +1,7 @@
 <?xml version="1.0"?>
 <robot name="ieg76" xmlns:xacro="http://www.ros.org/wiki/xacro">
-    <material name="ieg76-metal">
-        <color rgba="0.5 0.45 0.4 1"/>
-    </material>
-    <xacro:property name="base_x" value="0.112"/>
-    <xacro:property name="base_y" value="0.090"/>
-    <xacro:property name="base_z" value="0.08725"/>
-    <xacro:property name="jaw_base_y" value="0.0228"/>
-    <xacro:property name="jaw_base_z" value="0.0191"/>
+    <xacro:property name="base_x" value="0.060"/>
+    <xacro:property name="base_y" value="0.071"/>
+    <xacro:property name="base_z" value="0.062"/>
     <xacro:macro name="ieg76" params="parent prefix *origin">
         <joint name="${prefix}mount" type="fixed">
@@ -16,4 +11,8 @@
         </joint>
         <link name="${prefix}base">
+            <inertial>
+                <origin xyz="0 0 0" rpy="0 0 0"/>
+                <mass value="0.73"/>
+                <inertia ixx="0.01" ixy="0" ixz="0" iyy="0.01" iyz="0" izz="0.01" />
             <visual>
                 <geometry>
@@ -25,22 +24,8 @@
             </visual>
         </link>
-        <joint name="${prefix}jaw_mount" type="fixed">
-            <origin rpy="0 0 0" xyz="0 0 ${base_z + jaw_base_z}"/>
+        <joint name="jaw_position" type="prismatic">
             <parent link="${prefix}base"/>
-            <child link="${prefix}jaw_base"/>
-        </joint>
-        <link name="${prefix}jaw_base">
-            <visual>
-                <origin rpy="0 0 0" xyz="0 0 ${-jaw_base_z/2}"/>
-                <geometry>
-                    <box size="${base_x} ${jaw_base_y} ${jaw_base_z}"/>
-                </geometry>
-                <material name="ieg76-metal"/>
-            </visual>
-        </link>
-        <joint name="egl_position" type="prismatic">
-            <parent link="${prefix}jaw_base"/>
             <child link="${prefix}finger_right"/>
-            <origin rpy="0.0 0.0 ${pi}" xyz="0.0255 -0.0255 -0.018"/>
+            <origin rpy="0.0 0.0 ${pi}" xyz="0.0255 -0.0255 ${base_z}"/>
             <axis xyz="1 0 0"/>
             <limit effort="100.0" lower="-0.015" upper="0.026" velocity="100.0"/>
@@ -51,5 +36,5 @@
                     <xacro:insert_block name="mesh"/>
                 </geometry>
-                <material name="grey ">
+                <material name="grey">
                     <color rgba="0.5 0.5 0.5 1.0"/>
                 </material>
@@ -61,11 +46,11 @@
             </collision>
         </link>
-        <joint name="egl_position_mimic" type="prismatic">
-            <parent link="${prefix}jaw_base"/>
+        <joint name="jaw_position_mimic" type="prismatic">
+            <parent link="${prefix}base"/>
             <child link="${prefix}finger_left"/>
-            <origin rpy="0.0 0.0 0.0" xyz="-0.0255 0.0255 -0.018"/>
+            <origin rpy="0.0 0.0 0.0" xyz="-0.0255 0.0255 ${base_z}"/>
             <axis xyz="1 0 0"/>
             <limit effort="100.0" lower="-0.015" upper="0.026" velocity="100.0"/>
-            <mimic joint="egl_position" multiplier="1"/>
+            <mimic joint="jaw_position" multiplier="1"/>
         </joint>
         <link name="${prefix}finger_left">
@@ -74,5 +59,5 @@
                      <xacro:insert_block name="mesh"/>
                 </geometry>
-                <material name="grey ">
+                <material name="grey">
                     <color rgba="0.5 0.5 0.5 1.0"/>
                 </material>

Commit message: Fixed driver shutdown/restart bug. Added robot-gripper adapter. Scaled stl file.

File: urdf/ieg76.urdf.xacro (robot description, xacro)
@@ -15,10 +15,12 @@
                 <mass value="0.73"/>
                 <inertia ixx="0.01" ixy="0" ixz="0" iyy="0.01" iyz="0" izz="0.01" />
+            </inertial>
             <visual>
+                <origin xyz="0 0 0" rpy="${pi/2.0} 0 0"/>
                 <geometry>
                     <mesh filename="package://weiss_gripper_ieg76/meshes/ieg76.stl"/>
                 </geometry>
                 <material name="black">
-                    <color rgba="0.0 0.0 0.0 1.0"/>
+                    <color rgba="1 1 1 1.0"/>
                 </material>
             </visual>
@@ -34,5 +36,5 @@
             <visual>
                 <geometry>
-                    <xacro:insert_block name="mesh"/>
+                    <mesh filename="package://weiss_gripper_ieg76/meshes/finger.stl"/>
                 </geometry>
                 <material name="grey">
@@ -42,5 +44,5 @@
             <collision>
                 <geometry>
-                    <xacro:insert_block name="mesh"/>
+                    <mesh filename="package://weiss_gripper_ieg76/meshes/finger.stl"/>
                 </geometry>
             </collision>
@@ -57,5 +59,5 @@
             <visual>
                 <geometry>
-                     <xacro:insert_block name="mesh"/>
+                    <mesh filename="package://weiss_gripper_ieg76/meshes/finger.stl"/>
                 </geometry>
                 <material name="grey">
@@ -65,5 +67,5 @@
             <collision>
                 <geometry>
-                     <xacro:insert_block name="mesh"/>
+                    <mesh filename="package://weiss_gripper_ieg76/meshes/finger.stl"/>
                 </geometry>
             </collision>

Commit message: Updated readme file and removed fingers

File: urdf/ieg76.urdf.xacro (robot description, xacro)
@@ -33,19 +33,5 @@
             <limit effort="100.0" lower="-0.015" upper="0.026" velocity="100.0"/>
         </joint>
-        <link name="${prefix}finger_right">
-            <visual>
-                <geometry>
-                    <mesh filename="package://weiss_gripper_ieg76/meshes/finger.stl"/>
-                </geometry>
-                <material name="grey">
-                    <color rgba="0.5 0.5 0.5 1.0"/>
-                </material>
-            </visual>
-            <collision>
-                <geometry>
-                    <mesh filename="package://weiss_gripper_ieg76/meshes/finger.stl"/>
-                </geometry>
-            </collision>
-        </link>
+        <link name="${prefix}finger_right"/>
         <joint name="jaw_position_mimic" type="prismatic">
             <parent link="${prefix}base"/>
@@ -56,19 +42,5 @@
             <mimic joint="jaw_position" multiplier="1"/>
         </joint>
-        <link name="${prefix}finger_left">
-            <visual>
-                <geometry>
-                    <mesh filename="package://weiss_gripper_ieg76/meshes/finger.stl"/>
-                </geometry>
-                <material name="grey">
-                    <color rgba="0.5 0.5 0.5 1.0"/>
-                </material>
-            </visual>
-            <collision>
-                <geometry>
-                    <mesh filename="package://weiss_gripper_ieg76/meshes/finger.stl"/>
-                </geometry>
-            </collision>
-        </link>
+        <link name="${prefix}finger_left"/>
     </xacro:macro>
 </robot>

Commit message: add static grip center frame

File: urdf/ieg76.urdf.xacro (robot description, xacro)
@@ -43,4 +43,11 @@
         </joint>
         <link name="${prefix}finger_left"/>
+        <joint name="${prefix}center" type="fixed">
+            <parent link="${parent}"/>
+            <child link="${prefix}center"/>
+            <origin rpy="0 0 0" xyz="0 0 ${base_z}"/>
+        </joint>
+        <link name="${prefix}center">
+        </link>
     </xacro:macro>
 </robot>
