Commit message: ieg55 and new values for ieg76

File: urdf/ieg55.urdf.xacro (robot description, xacro)
@@ -1,5 +1,5 @@
 <?xml version="1.0"?>
-<robot name="ieg76" xmlns:xacro="http://www.ros.org/wiki/xacro">
-    <xacro:macro name="ieg76" params="parent prefix *origin">
+<robot name="ieg55" xmlns:xacro="http://www.ros.org/wiki/xacro">
+    <xacro:macro name="ieg55" params="parent prefix *origin">
         <joint name="${prefix}mount" type="fixed">
             <insert_block name="origin"/>
@@ -10,11 +10,10 @@
             <inertial>
                 <origin xyz="0 0 0" rpy="0 0 0"/>
-                <mass value="0.73"/>
+                <mass value="0.27"/>
                 <inertia ixx="0.01" ixy="0" ixz="0" iyy="0.01" iyz="0" izz="0.01" />
             </inertial>
             <visual>
-                <origin xyz="0 0 0" rpy="${pi/2.0} 0 0"/>
                 <geometry>
-                    <mesh filename="package://weiss_gripper_ieg76/meshes/ieg76.stl"/>
+                    <mesh filename="package://weiss_gripper_ieg76/meshes/ieg55.stl"/>
                 </geometry>
                 <material name="black">
@@ -26,7 +25,7 @@
             <parent link="${prefix}base"/>
             <child link="${prefix}finger_right"/>
-            <origin rpy="0.0 0.0 ${pi}" xyz="0.0 -0.0185 0.063"/>
+            <origin rpy="0.0 0.0 ${pi}" xyz="0.0 -0.0115 0.045"/>
             <axis xyz="1 0 0"/>
-            <limit effort="100.0" lower="0.0" upper="0.015" velocity="100.0"/>
+            <limit effort="100.0" lower="0.0" upper="0.01" velocity="100.0"/>
         </joint>
         <link name="${prefix}finger_right"/>
@@ -34,7 +33,7 @@
             <parent link="${prefix}base"/>
             <child link="${prefix}finger_left"/>
-            <origin rpy="0.0 0.0 0.0" xyz="0.0 0.0185 0.063"/>
+            <origin rpy="0.0 0.0 0.0" xyz="0.0 0.0115 0.045"/>
             <axis xyz="1 0 0"/>
-            <limit effort="100.0" lower="0.0" upper="0.015" velocity="100.0"/>
+            <limit effort="100.0" lower="0.0" upper="0.01" velocity="100.0"/>
             <mimic joint="jaw_position" multiplier="1"/>
         </joint>
@@ -43,5 +42,5 @@
             <parent link="${parent}"/>
             <child link="${prefix}center"/>
-            <origin rpy="0 0 0" xyz="0 0 0.063"/>
+            <origin rpy="0 0 0" xyz="0 0 0.045"/>
         </joint>
         <link name="${prefix}center"/>

File: urdf/ieg55_adapter.urdf.xacro (robot description, xacro)
@@ -1,5 +1,5 @@
 <?xml version="1.0"?>
-<robot xmlns:xacro="http://www.ros.org/wiki/xacro" name="ieg76_adapter">
-    <xacro:macro name="ieg76_adapter" params="parent prefix *origin">
+<robot xmlns:xacro="http://www.ros.org/wiki/xacro" name="ieg55_adapter">
+    <xacro:macro name="ieg55_adapter" params="parent prefix *origin">
         <!-- mount the adapter to the robot -->
         <joint name="${prefix}robotside_joint" type="fixed">
@@ -12,5 +12,5 @@
                 <origin xyz="0 0 0.005" rpy="0 0 0"/>
                 <geometry>
-                    <box size="0.076 0.06 0.01"/>
+                    <box size="0.055 0.041 0.01"/>
                 </geometry>
                 <material name="metal">
@@ -21,5 +21,5 @@
                 <origin xyz="0 0 0.005" rpy="0 0 0"/>
                 <geometry>
-                    <box size="0.076 0.06 0.01"/>
+                    <box size="0.055 0.041 0.01"/>
                 </geometry>
             </collision>

Commit message: FIX: prefixes for multiple instances

File: urdf/ieg55.urdf.xacro (robot description, xacro)
@@ -22,5 +22,5 @@
             </visual>
         </link>
-        <joint name="jaw_position" type="prismatic">
+        <joint name="${prefix}jaw_position" type="prismatic">
             <parent link="${prefix}base"/>
             <child link="${prefix}finger_right"/>
@@ -30,5 +30,5 @@
         </joint>
         <link name="${prefix}finger_right"/>
-        <joint name="jaw_position_mimic" type="prismatic">
+        <joint name="${prefix}jaw_position_mimic" type="prismatic">
             <parent link="${prefix}base"/>
             <child link="${prefix}finger_left"/>
@@ -36,8 +36,8 @@
             <axis xyz="1 0 0"/>
             <limit effort="100.0" lower="0.0" upper="0.01" velocity="100.0"/>
-            <mimic joint="jaw_position" multiplier="1"/>
+            <mimic joint="${prefix}jaw_position" multiplier="1"/>
         </joint>
         <link name="${prefix}finger_left"/>
-        <joint name="${prefix}center" type="fixed">
+        <joint name="${prefix}${prefix}center" type="fixed">
             <parent link="${parent}"/>
             <child link="${prefix}center"/>

File: urdf/ieg76.urdf.xacro (robot description, xacro)
@@ -2,5 +2,5 @@
 <robot name="ieg76" xmlns:xacro="http://www.ros.org/wiki/xacro">
     <xacro:macro name="ieg76" params="parent prefix *origin">
-        <joint name="${prefix}mount" type="fixed">
+        <joint name="$${prefix}mount" type="fixed">
             <insert_block name="origin"/>
             <parent link="${parent}"/>
@@ -23,5 +23,5 @@
             </visual>
         </link>
-        <joint name="jaw_position" type="prismatic">
+        <joint name="${prefix}jaw_position" type="prismatic">
             <parent link="${prefix}base"/>
             <child link="${prefix}finger_right"/>
@@ -31,5 +31,5 @@
         </joint>
         <link name="${prefix}finger_right"/>
-        <joint name="jaw_position_mimic" type="prismatic">
+        <joint name="${prefix}jaw_position_mimic" type="prismatic">
             <parent link="${prefix}base"/>
             <child link="${prefix}finger_left"/>
@@ -37,5 +37,5 @@
             <axis xyz="1 0 0"/>
             <limit effort="100.0" lower="0.0" upper="0.015" velocity="100.0"/>
-            <mimic joint="jaw_position" multiplier="1"/>
+            <mimic joint="${prefix}jaw_position" multiplier="1"/>
         </joint>
         <link name="${prefix}finger_left"/>

Commit message: todo: separate into different commits (working on checking serial no)

File: urdf/ieg55.urdf.xacro (robot description, xacro)
@@ -22,5 +22,5 @@
             </visual>
         </link>
-        <joint name="${prefix}jaw_position" type="prismatic">
+        <!-- <joint name="${prefix}jaw_position" type="prismatic">
             <parent link="${prefix}base"/>
             <child link="${prefix}finger_right"/>
@@ -38,5 +38,5 @@
             <mimic joint="${prefix}jaw_position" multiplier="1"/>
         </joint>
-        <link name="${prefix}finger_left"/>
+        <link name="${prefix}finger_left"/> -->
         <joint name="${prefix}${prefix}center" type="fixed">
             <parent link="${parent}"/>

Commit message: fixed urdf

File: urdf/ieg55.urdf.xacro (robot description, xacro)
@@ -39,5 +39,5 @@
         </joint>
         <link name="${prefix}finger_left"/> -->
-        <joint name="${prefix}${prefix}center" type="fixed">
+        <joint name="${prefix}center" type="fixed">
             <parent link="${parent}"/>
             <child link="${prefix}center"/>

File: urdf/ieg76.urdf.xacro (robot description, xacro)
@@ -2,5 +2,5 @@
 <robot name="ieg76" xmlns:xacro="http://www.ros.org/wiki/xacro">
     <xacro:macro name="ieg76" params="parent prefix *origin">
-        <joint name="$${prefix}mount" type="fixed">
+        <joint name="${prefix}mount" type="fixed">
             <insert_block name="origin"/>
             <parent link="${parent}"/>
